Commit message: Drive wheels: sphere collision, so they touch the ground in their center plane
With a collision cylinder and minDepth 0, Remo turned only 1.28 of 1.50 rad on the
spot in the simulation test, the ratio of its wheel separation to the distance
between the wheels' outer edges (0.144 / 0.169 m). A sphere with the wheel radius
touches the ground at one point in the wheel's center plane, as DiffBot's does since
diffbot#120.

fdir1 is removed: Gazebo turns it with the collision frame, and a sphere's frame spins
with the wheel. With fdir1 0 0 1, Remo slipped 1.7 % driving straight.

File: urdf/include/common_macros.urdf.xacro (robot description, xacro)
@@ -46,8 +46,12 @@
       </visual>
     </xacro:if>
+      <!-- Use a sphere with the wheel radius for collision. On flat ground, an upright wheel's
+           contact stays in its center plane. This avoids the outer-edge cylinder contacts that
+           can increase the effective wheel separation and reduce the true turn relative to
+           odometry. The wheel visual and cylinder inertia are unchanged.
+           See https://github.com/ros-mobile-robots/remo_description/pull/2 -->
       <collision>
-        <origin xyz="0 0 0" rpy="${pi/2} 0 0"/>
-        <geometry>
-          <cylinder radius="${wheel_props['radius']}" length="${wheel_props['length']}"/>
+        <geometry>
+          <sphere radius="${wheel_props['radius']}"/>
         </geometry>
       </collision>

File: urdf/include/robot.gazebo.xacro (robot description, xacro)
@@ -36,5 +36,7 @@
     <!-- Use moderate friction and compliant, damped drive-wheel contacts to limit Remo's
          stick-slip jitter when turning in Gazebo. Reuse the friction argument and kp/kd
-         settings from set_wheel_friction above.
+         settings from set_wheel_friction above. Leave fdir1 unset: Gazebo turns it with the
+         collision frame, which spins with the wheel's sphere collision, so it would tilt into
+         the contact normal and make the wheels slip.
          See https://github.com/ros-mobile-robots/remo_description/pull/2 -->
     <gazebo reference="front_right_wheel">
@@ -45,5 +47,4 @@
       <minDepth>0.01</minDepth>      <!-- minimum allowable depth before contact correction impulse is applied (default 0) -->
       <maxVel>0.01</maxVel> <!-- maximum contact correction velocity truncation term (default 0.01)-->
-      <fdir1>0 0 1</fdir1>   <!-- 3-tuple specifying direction of mu1 in the collision local reference frame (default 0 0 0) -->
       <material>Gazebo/FlatBlack</material>
     </gazebo>
@@ -55,5 +56,4 @@
       <minDepth>0.01</minDepth>
       <maxVel>0.01</maxVel>
-      <fdir1>0 0 1</fdir1>
       <material>Gazebo/FlatBlack</material>
     </gazebo>

Commit message: Frames: base_link and base_footprint at the axle's midpoint
diff_drive_controller computes the odometry for the midpoint between the drive
wheels and publishes it as base_footprint. That frame was below the center of
the base plate, 36 mm behind the axle, so during a turn on the spot TF put the
robot and its sensors on a small arc that the real robot doesn't drive.

base_link is now the axle's midpoint, with base_footprint on the ground below
it, as before. The base plate's geometry and mass, and every part attached to
it, are defined around a new chassis_link, 36 mm behind base_link, so no part
moves relative to the others. The offset comes from the existing base size and
wheel offset, the same values the wheel joint uses.

File: urdf/include/common_macros.urdf.xacro (robot description, xacro)
@@ -68,5 +68,5 @@
     <joint name="${prefix}_wheel_joint" type="continuous">
       <axis xyz="0 1 0" rpy="0 0 0" />
-      <parent link="base_link"/>
+      <parent link="chassis_link"/>
       <child link="${prefix}_wheel"/>
       <origin xyz="${pos_x_joint} ${reflect* pos_y_joint} ${pos_z_joint}" rpy="0 0 0"/>
@@ -138,5 +138,5 @@
     </link>
     <joint name="${prefix}_motor_joint" type="fixed">
-      <parent link="base_link"/>
+      <parent link="chassis_link"/>
       <child link="${prefix}_motor"/>
       <origin xyz="${pos_x_joint} ${reflect* pos_y_joint} ${pos_z_joint}" rpy="0 ${-pi/2.0*(reflect - 1)} 0"/>

File: urdf/include/remo_base_macro.urdf.xacro (robot description, xacro)
@@ -6,4 +6,6 @@
   params:
   - base_props [dictionary]: base link properties;
+  - axle_x [float]: how far the drive axle's midpoint (base_link) lies in front of the base
+    plate's center (chassis_link), in m;
   - mesh [string]: file name of the link mesh;
     - DEFAULT Value -> Empty string
@@ -11,6 +13,16 @@
 -->
   <xacro:macro name="base"
-               params="base_prop mesh:='' scale:='' *origin ">
-    <link name="base_link">
+               params="base_prop axle_x mesh:='' scale:='' *origin ">
+    <!-- base_link is the robot's reference frame: the midpoint between the drive wheels, where
+         diff_drive_controller's odometry puts the robot. The chassis' geometry, mass and all
+         attached parts are defined around chassis_link, the center of the base plate, which lies
+         axle_x behind it. -->
+    <link name="base_link" />
+    <joint name="chassis_joint" type="fixed">
+      <parent link="base_link"/>
+      <child link="chassis_link"/>
+      <origin xyz="${-axle_x} 0 0" rpy="0 0 0"/>
+    </joint>
+    <link name="chassis_link">
     <xacro:box_inertia m="${base_prop['base']['mass']}"
                        x="${base_prop['base']['x_size']}"
@@ -50,5 +62,5 @@
     </collision>
     </link>
-    <gazebo reference="base_link">
+    <gazebo reference="chassis_link">
       <material>Gazebo/Grey</material>
     </gazebo>

File: urdf/include/remo_caster_macro.urdf.xacro (robot description, xacro)
@@ -57,5 +57,5 @@
       <origin xyz="${wheel_props['base']['dx']} ${-wheel_props['base']['dy'] * locationright} ${wheel_props['base']['dz']}"
               rpy="0 0 0" />
-      <parent link="base_link" />
+      <parent link="chassis_link" />
       <child link="${prefix}_caster_base_link" />
     </joint>
@@ -104,5 +104,5 @@
       <origin xyz="${wheel_props['hub']['dx']} ${-wheel_props['hub']['dy'] * locationright} ${wheel_props['hub']['dz']}"
               rpy="0 0 0" />
-      <parent link="base_link" />
+      <parent link="chassis_link" />
       <child link="${prefix}_caster_rotation_link" />
       <axis xyz="0 0 1" />

File: urdf/remo.urdf.xacro (robot description, xacro)
@@ -29,6 +29,8 @@
   <!-- Footprint link -->
   <xacro:footprint wheel_props="${front_wheel_props}" />
-  <!-- Base link -->
-  <xacro:base base_prop="${base_props}" mesh="${base_props['base']['mesh']}" scale="0.001 0.001 0.001">
+  <!-- Base link at the drive axle's midpoint, and the chassis around it. The wheels sit
+       x_offset behind the base plate's front edge, the same position the wheel macro uses -->
+  <xacro:property name="axle_x" value="${base_props['base']['x_size']/2 - front_wheel_props['x_offset']}"/>
+  <xacro:base base_prop="${base_props}" axle_x="${axle_x}" mesh="${base_props['base']['mesh']}" scale="0.001 0.001 0.001">
     <origin xyz="0 0 0" rpy="0 0 0" />
   </xacro:base>
@@ -59,5 +61,5 @@
     <xacro:property name="deck_type" value="'jetson_deck'"/>
     <!-- Deck link -->
-    <xacro:addon addon="jetson_deck" base_prop="${base_props}" parent_link="base_link" >
+    <xacro:addon addon="jetson_deck" base_prop="${base_props}" parent_link="chassis_link" >
       <origin xyz="0 0 0" rpy="0 0 0" />
     </xacro:addon>
@@ -67,5 +69,5 @@
     </xacro:addon>
     <!-- Breadboard 400 point -->
-    <xacro:addon addon="breadboard" base_prop="${component_props}" parent_link="base_link" >
+    <xacro:addon addon="breadboard" base_prop="${component_props}" parent_link="chassis_link" >
       <origin xyz="-0.05 0 0" rpy="0 0 0" />
     </xacro:addon>
@@ -74,5 +76,5 @@
     <xacro:property name="deck_type" value="'rpi_deck'"/>
     <!-- Deck link -->
-    <xacro:addon addon="rpi_deck" base_prop="${base_props}" parent_link="base_link" >
+    <xacro:addon addon="rpi_deck" base_prop="${base_props}" parent_link="chassis_link" >
       <origin xyz="0 0 0" rpy="0 0 0" />
     </xacro:addon>
@@ -82,5 +84,5 @@
     </xacro:addon>
     <!-- Breadboard 400 point -->
-    <xacro:addon addon="breadboard" base_prop="${component_props}" parent_link="base_link" >
+    <xacro:addon addon="breadboard" base_prop="${component_props}" parent_link="chassis_link" >
       <origin xyz="-0.04 0 0" rpy="0 0 0" />
     </xacro:addon>
@@ -106,5 +108,5 @@
   <!-- Camera -->
   <!-- Camera mount link -->
-  <xacro:addon addon="camera_mount" base_prop="${base_props}" parent_link="base_link" >
+  <xacro:addon addon="camera_mount" base_prop="${base_props}" parent_link="chassis_link" >
     <origin xyz="0.085198 0 -0.0081709" rpy="0 0 0" />
   </xacro:addon>
@@ -148,5 +150,5 @@
   </xacro:if>
   <!-- IMU
-  <xacro:imu_sensor parent_link="base_link"
+  <xacro:imu_sensor parent_link="chassis_link"
                     sensor_prop="${sensor_props}">
     <origin xyz="-0.045 0.02 0.01" rpy="0 0 0" />
@@ -159,14 +161,14 @@
   </xacro:set_all_wheel_frictions>
   <!-- Additional addons -->
-  <xacro:addon addon="power_bank" base_prop="${component_props}" parent_link="base_link" >
+  <xacro:addon addon="power_bank" base_prop="${component_props}" parent_link="chassis_link" >
     <origin xyz="0 0 -0.01" rpy="0 0 0" />
   </xacro:addon>
-  <xacro:addon addon="battery_pack" base_prop="${component_props}" parent_link="base_link" >
+  <xacro:addon addon="battery_pack" base_prop="${component_props}" parent_link="chassis_link" >
     <origin xyz="0.045 0 -0.04" rpy="0 0 0" />
   </xacro:addon>
-  <xacro:addon addon="mcu" base_prop="${component_props}" parent_link="base_link" >
+  <xacro:addon addon="mcu" base_prop="${component_props}" parent_link="chassis_link" >
     <origin xyz="-0.045 -0.02 0.01" rpy="0 0 ${-pi/2}" />
   </xacro:addon>
-  <xacro:addon addon="motor_driver" base_prop="${component_props}" parent_link="base_link" >
+  <xacro:addon addon="motor_driver" base_prop="${component_props}" parent_link="chassis_link" >
     <origin xyz="-0.0086 0 -0.0277" rpy="0 0 0" />
   </xacro:addon>
