Commit message: Frames: base_link and base_footprint at the axle's midpoint (#5)
`base_link` is now directly above the midpoint between the drive wheels, at the same height as before, with `base_footprint` on the ground below it. The base plate's geometry and mass, and every part attached to it, hang off a new `chassis_link`, 36 mm behind `base_link`.

**Why:** `diff_drive_controller` computes the odometry for the axle's midpoint and publishes it as `base_footprint`. But in the URDF, `base_footprint` was on the ground under the center of the base plate, and that center is 36 mm behind the axle. The controller's odometry and the URDF used different reference points, so TF placed the chassis and the sensors incorrectly during turns (ros-mobile-robots/diffbot#118).

**Other robots:** TurtleBot3 Burger and Linorobot2 also put `base_link` at the axle's midpoint in x and y. They have no `chassis_link`: they attach the body and the other parts to `base_link` directly.
- **TurtleBot3 Burger:** the wheel joints are at x = 0 in `base_link` ([line 42](https://github.com/ROBOTIS-GIT/turtlebot3/blob/4ae959ea6a52415c90bf752d2b76e3e28f8a87e2/turtlebot3_description/urdf/turtlebot3_burger.urdf.xacro#L42)). The body's visual and collision are shifted 32 mm back inside `base_link` ([line 16](https://github.com/ROBOTIS-GIT/turtlebot3/blob/4ae959ea6a52415c90bf752d2b76e3e28f8a87e2/turtlebot3_description/urdf/turtlebot3_burger.urdf.xacro#L16), [line 24](https://github.com/ROBOTIS-GIT/turtlebot3/blob/4ae959ea6a52415c90bf752d2b76e3e28f8a87e2/turtlebot3_description/urdf/turtlebot3_burger.urdf.xacro#L24)).
- **Linorobot2 (2WD):** the wheels are at `wheel_pos_x` 0.0 ([2wd_properties, line 13](https://github.com/linorobot/linorobot2/blob/f6b0bd0350c4a9d6b815ef4bb5c701a1e5129711/linorobot2_description/urdf/2wd_properties.urdf.xacro#L13)), and the body is centered on `base_link` ([base.urdf.xacro, lines 6–36](https://github.com/linorobot/linorobot2/blob/f6b0bd0350c4a9d6b815ef4bb5c701a1e5129711/linorobot2_description/urdf/mech/base.urdf.xacro#L6-L36)).
- **Clearpath's Jackal** separates the two frames the same way, and `chassis_link` is its name: an empty `base_link` with a fixed joint to `chassis_link`, which holds the body. Its joint is zero, because Jackal's four wheels sit symmetrically around the body's center ([jackal.urdf.xacro, lines 82–103](https://github.com/jackal/jackal/blob/4ddf9b578bb7abce1115c8dc59d8b7f86aa9268c/jackal_description/urdf/jackal.urdf.xacro#L82-L103)). On Remo, the axle is 36 mm in front of the plate's center, so the joint holds those 36 mm.

Remo's parts are given from the plate's center instead. Without `chassis_link`, the plate's geometry and every part's attachment point would have to be given from `base_link` at the axle: their x values change by 36 mm, in 14 places in the xacro and YAML files (counting both `sbc_type` variants and the disabled IMU). The parts themselves don't move. With `chassis_link`, one fixed joint holds the 36 mm, and the parts keep their numbers. Both ways give the same model: the frames they share have the same poses in TF, and Gazebo Classic's default URDF conversion merges these fixed links into one body.

**Height of `base_link`:** unchanged. `base_link` is at the top of the base plate's box, 66.6 mm above the ground: the wheel radius, 33.0 mm from the ground to the axle, plus 33.6 mm from the axle up to `base_link`. [`front_wheel.yaml`](https://github.com/ros-mobile-robots/remo_description/blob/055b07564ec8c34c79adaf53175c0317b2b113cd/config/remo/front_wheel.yaml#L2-L9) gives these as `radius: 0.0330` and `z_offset: -0.0336` (the axle is below `base_link`, so it's negative), and `base_footprint` → `base_link` is `radius − z_offset` ([`common_macros.urdf.xacro`, line 245](https://github.com/ros-mobile-robots/remo_description/blob/055b07564ec8c34c79adaf53175c0317b2b113cd/urdf/include/common_macros.urdf.xacro#L245)). Only x changes: `base_link` and `base_footprint` move 36 mm forward, from the plate's center to the axle. ROS's frame convention, [REP 105](https://www.ros.org/reps/rep-0105.html#base-link), leaves the place of `base_link` to each robot.

<img width="1080" height="1110" alt="side-view-5" src="https://github.com/user-attachments/assets/ca40beff-9dff-4a12-a8b5-b2d139527316" />


**What changes:**
- `remo_base_macro.urdf.xacro`: the macro creates an empty `base_link`, a fixed `chassis_joint` and `chassis_link` with the plate's visual, collision and inertia, unchanged. The offset `axle_x` (36 mm, from the plate's center to the axle) comes from the plate's length and the wheels' `x_offset` (34 mm, from the plate's front edge to the axle): `axle_x` = 140 / 2 − 34 mm. The wheel joint uses the same values, so `axle_x` follows them if they change.
- The wheels, motors, caster and all add-ons attach to `chassis_link` instead of `base_link`, with their joint origins unchanged.

## Link tree

Remo with the default `sbc_type` (`rpi`) and `camera_type` (`raspi-cam`). Before this change, `base_link` was the plate's center and every part hung off it. Now `chassis_link` (highlighted) holds the plate, 36 mm behind `base_link`, and the parts hang off it with unchanged joint origins.

```mermaid
graph TB
  fp[base_footprint] -->|"z +66.6 mm"| bl[base_link]
  bl -->|"x −36 mm"| ch[chassis_link]
  ch --> wl[front_left_wheel]
  ch --> wr[front_right_wheel]
  ch --> ml[left_motor]
  ch --> mr[right_motor]
  ch --> cb[rear_caster_base_link]
  ch --> cr[rear_caster_rotation_link] --> cw[rear_caster_wheel_link]
  ch --> deck[rpi_deck_link]
  deck --> rpi[rpi_link]
  deck --> lp[lidar_platform_link]
  lp --> sh[slamtec_holder_link] --> usb[slamtec_usb_to_serial_link]
  lp --> laser[rplidar_laser_link]
  ch --> cm[camera_mount_link] --> rc["raspi-cam_link"] --> cam[camera_link]
  ch --> bb[breadboard_link]
  ch --> pb[power_bank_link]
  ch --> bp[battery_pack_link]
  ch --> mcu[mcu_link]
  ch --> md[motor_driver_link]
  classDef new fill:#fff3c4,stroke:#c79a00,color:#000
  class ch new
```

**Version and merge order:** this moves `base_link`, so things built on the model have to change too: the version goes from 1.0.0 to 2.0.0, in `package.xml` and a new `CHANGELOG.rst` section. diffbot's workspace pins version 1.0.0 (ros-mobile-robots/diffbot#129), so merging this doesn't change diffbot until the pin moves. After the merge, the merge commit gets the tag `2.0.0`, and ros-mobile-robots/diffbot#130 moves the pin to it. #130 adapts diffbot: DiffBot's frames, both robots' navigation footprints and the simulation test. The Insiders repository, which has the meshes, gets the same change and tag.

## How it was checked

- Expanded URDFs, old (e6232d0, the same model as 1.0.0) and new, for every `sbc_type` and `camera_type`: each link's pose relative to the chassis is unchanged; only `base_link` and `base_footprint` move, 36 mm forward. The wheel joints are at x = 0 in `base_link`, and `base_footprint` → `base_link` is unchanged (0.0666 m).
- For comparison, a variant without `chassis_link`, with the plate and every part's attachment point given from `base_link` instead: for every `sbc_type` and `camera_type`, each link and its visual, collision and inertia are at the same pose as with `chassis_link`.
- The simulation test in diffbot's dev container image, two runs with diffbot `noetic-devel`: all 10 tests pass. During the turn on the spot, Remo's true pose now moves 0.000 m instead of 0.033 m forward and 0.036 m sideways; straight driving is unchanged (0.580 m). Three more runs with ros-mobile-robots/diffbot#130 (both robots at the axle): all pass, Remo's turn again 0.000 m.
- Rebased onto `main` (version 1.0.0): the expanded URDFs of all six variants are byte-identical to the ones before the rebase, so the checks above still apply. `catkin_pkg` reads the package as version 2.0.0 and parses both changelog sections.

File: urdf/include/remo_base_macro.urdf.xacro (robot description, xacro)
@@ -6,4 +6,6 @@
   params:
   - base_props [dictionary]: base link properties;
+  - axle_x [float]: how far the drive axle's midpoint (base_link) lies in front of the base
+    plate's center (chassis_link), in m;
   - mesh [string]: file name of the link mesh;
     - DEFAULT Value -> Empty string
@@ -11,6 +13,16 @@
 -->
   <xacro:macro name="base"
-               params="base_prop mesh:='' scale:='' *origin ">
-    <link name="base_link">
+               params="base_prop axle_x mesh:='' scale:='' *origin ">
+    <!-- base_link is the robot's reference frame: the midpoint between the drive wheels, where
+         diff_drive_controller's odometry puts the robot. chassis_link is the center of the base
+         plate, axle_x behind base_link. The plate's geometry and mass, and all parts attached to
+         it, are defined around chassis_link. -->
+    <link name="base_link" />
+    <joint name="chassis_joint" type="fixed">
+      <parent link="base_link"/>
+      <child link="chassis_link"/>
+      <origin xyz="${-axle_x} 0 0" rpy="0 0 0"/>
+    </joint>
+    <link name="chassis_link">
     <xacro:box_inertia m="${base_prop['base']['mass']}"
                        x="${base_prop['base']['x_size']}"
@@ -50,5 +62,5 @@
     </collision>
     </link>
-    <gazebo reference="base_link">
+    <gazebo reference="chassis_link">
       <material>Gazebo/Grey</material>
     </gazebo>

File: urdf/remo.urdf.xacro (robot description, xacro)
@@ -29,6 +29,10 @@
   <!-- Footprint link -->
   <xacro:footprint wheel_props="${front_wheel_props}" />
-  <!-- Base link -->
-  <xacro:base base_prop="${base_props}" mesh="${base_props['base']['mesh']}" scale="0.001 0.001 0.001">
+  <!-- Base link at the drive axle's midpoint, and the chassis around it. axle_x is how far the
+       axle is in front of the plate's center. The wheel config gives the axle's position from the
+       plate's front edge instead (x_offset), so axle_x = half the plate's length - x_offset
+       (0.070 - 0.034 = 0.036 m). The wheel macro places the wheels with the same formula. -->
+  <xacro:property name="axle_x" value="${base_props['base']['x_size']/2 - front_wheel_props['x_offset']}"/>
+  <xacro:base base_prop="${base_props}" axle_x="${axle_x}" mesh="${base_props['base']['mesh']}" scale="0.001 0.001 0.001">
     <origin xyz="0 0 0" rpy="0 0 0" />
   </xacro:base>
@@ -59,5 +63,5 @@
     <xacro:property name="deck_type" value="'jetson_deck'"/>
     <!-- Deck link -->
-    <xacro:addon addon="jetson_deck" base_prop="${base_props}" parent_link="base_link" >
+    <xacro:addon addon="jetson_deck" base_prop="${base_props}" parent_link="chassis_link" >
       <origin xyz="0 0 0" rpy="0 0 0" />
     </xacro:addon>
@@ -67,5 +71,5 @@
     </xacro:addon>
     <!-- Breadboard 400 point -->
-    <xacro:addon addon="breadboard" base_prop="${component_props}" parent_link="base_link" >
+    <xacro:addon addon="breadboard" base_prop="${component_props}" parent_link="chassis_link" >
       <origin xyz="-0.05 0 0" rpy="0 0 0" />
     </xacro:addon>
@@ -74,5 +78,5 @@
     <xacro:property name="deck_type" value="'rpi_deck'"/>
     <!-- Deck link -->
-    <xacro:addon addon="rpi_deck" base_prop="${base_props}" parent_link="base_link" >
+    <xacro:addon addon="rpi_deck" base_prop="${base_props}" parent_link="chassis_link" >
       <origin xyz="0 0 0" rpy="0 0 0" />
     </xacro:addon>
@@ -82,5 +86,5 @@
     </xacro:addon>
     <!-- Breadboard 400 point -->
-    <xacro:addon addon="breadboard" base_prop="${component_props}" parent_link="base_link" >
+    <xacro:addon addon="breadboard" base_prop="${component_props}" parent_link="chassis_link" >
       <origin xyz="-0.04 0 0" rpy="0 0 0" />
     </xacro:addon>
@@ -106,5 +110,5 @@
   <!-- Camera -->
   <!-- Camera mount link -->
-  <xacro:addon addon="camera_mount" base_prop="${base_props}" parent_link="base_link" >
+  <xacro:addon addon="camera_mount" base_prop="${base_props}" parent_link="chassis_link" >
     <origin xyz="0.085198 0 -0.0081709" rpy="0 0 0" />
   </xacro:addon>
@@ -148,5 +152,5 @@
   </xacro:if>
   <!-- IMU
-  <xacro:imu_sensor parent_link="base_link"
+  <xacro:imu_sensor parent_link="chassis_link"
                     sensor_prop="${sensor_props}">
     <origin xyz="-0.045 0.02 0.01" rpy="0 0 0" />
@@ -159,14 +163,14 @@
   </xacro:set_all_wheel_frictions>
   <!-- Additional addons -->
-  <xacro:addon addon="power_bank" base_prop="${component_props}" parent_link="base_link" >
+  <xacro:addon addon="power_bank" base_prop="${component_props}" parent_link="chassis_link" >
     <origin xyz="0 0 -0.01" rpy="0 0 0" />
   </xacro:addon>
-  <xacro:addon addon="battery_pack" base_prop="${component_props}" parent_link="base_link" >
+  <xacro:addon addon="battery_pack" base_prop="${component_props}" parent_link="chassis_link" >
     <origin xyz="0.045 0 -0.04" rpy="0 0 0" />
   </xacro:addon>
-  <xacro:addon addon="mcu" base_prop="${component_props}" parent_link="base_link" >
+  <xacro:addon addon="mcu" base_prop="${component_props}" parent_link="chassis_link" >
     <origin xyz="-0.045 -0.02 0.01" rpy="0 0 ${-pi/2}" />
   </xacro:addon>
-  <xacro:addon addon="motor_driver" base_prop="${component_props}" parent_link="base_link" >
+  <xacro:addon addon="motor_driver" base_prop="${component_props}" parent_link="chassis_link" >
     <origin xyz="-0.0086 0 -0.0277" rpy="0 0 0" />
   </xacro:addon>
