Commit message: IMU: imu_link for the BNO055 with a Gazebo IMU sensor
Remo's model gets imu_link, the BNO055 board on chassis_link, and a Gazebo IMU sensor (gazebo_plugins' ROS 1 IMU plugin) that publishes /diffbot/imu/gazebo at 50 Hz, the firmware's rate. Its position is provisional: the earlier commented-out IMU's, with the board's axes along the robot's, as the xacro arguments imu_xyz and imu_rpy, until the board's mounting on the robot is confirmed. Version 2.1.0.

File: urdf/include/common_sensors.xacro (robot description, xacro)
@@ -175,3 +175,64 @@
   </gazebo>
 </xacro:macro>
+<!-- IMU: a Bosch BNO055 board, as a small box (sensor_prop['imu']: mass, size, mesh), and a Gazebo
+     IMU sensor that stands in for the real one in the simulation.
+     - imu_link is the sensor's own frame; *origin places it on parent_link, as the board sits on
+       the robot. The real robot's firmware publishes in the same frame (diffbot_base).
+     - The Gazebo plugin (gazebo_plugins' GazeboRosImuSensor, ROS 1) publishes sensor_msgs/Imu on
+       /diffbot/imu/gazebo at 50 Hz, the firmware's rate. Its message includes an orientation that
+       the real sensor doesn't provide, so the simulation passes it through an adapter in
+       diffbot_gazebo, which publishes /diffbot/imu/data_raw like the firmware.
+     - gaussianNoise is one standard deviation that the plugin adds to every value; it's a
+       simulation setting, not the BNO055's measured noise. -->
+<xacro:macro name="imu_sensor" params="parent_link sensor_prop *origin">
+  <xacro:property name="imu" value="${sensor_prop['imu']}"/>
+  <link name="imu_link">
+    <xacro:if value="${imu['mesh'] != ''}">
+      <visual>
+        <origin xyz="0 0 0" rpy="0 0 0"/>
+        <geometry>
+          <mesh filename="package://${package_name}/meshes/sensors/${imu['mesh']}" scale="${imu['scale']}"/>
+        </geometry>
+        <material name="dark_grey"/>
+      </visual>
+    </xacro:if>
+    <xacro:if value="${imu['mesh'] == ''}">
+      <visual>
+        <origin xyz="0 0 0" rpy="0 0 0"/>
+        <geometry>
+          <box size="${imu['size']['x']} ${imu['size']['y']} ${imu['size']['z']}"/>
+        </geometry>
+        <material name="red"/>
+      </visual>
+    </xacro:if>
+    <collision>
+      <origin xyz="0 0 0" rpy="0 0 0"/>
+      <geometry>
+        <box size="${imu['size']['x']} ${imu['size']['y']} ${imu['size']['z']}"/>
+      </geometry>
+    </collision>
+    <xacro:box_inertia m="${imu['mass']}" x="${imu['size']['x']}" y="${imu['size']['y']}" z="${imu['size']['z']}"/>
+  </link>
+  <joint name="imu_joint" type="fixed">
+    <parent link="${parent_link}"/>
+    <child link="imu_link"/>
+    <xacro:insert_block name="origin"/>
+  </joint>
+  <gazebo reference="imu_link">
+    <sensor type="imu" name="imu">
+      <always_on>true</always_on>
+      <update_rate>50</update_rate>
+      <plugin name="imu_plugin" filename="libgazebo_ros_imu_sensor.so">
+        <robotNamespace>/diffbot</robotNamespace>
+        <topicName>imu/gazebo</topicName>
+        <frameName>imu_link</frameName>
+        <updateRateHZ>50</updateRateHZ>
+        <gaussianNoise>0.005</gaussianNoise>
+        <xyzOffset>0 0 0</xyzOffset>
+        <rpyOffset>0 0 0</rpyOffset>
+        <initialOrientationAsReference>false</initialOrientationAsReference>
+      </plugin>
+    </sensor>
+  </gazebo>
+</xacro:macro>
 </robot>

File: urdf/remo.urdf.xacro (robot description, xacro)
@@ -7,4 +7,10 @@
   <!-- Must be one of ['rpi', 'jetson'] -->
   <xacro:arg name="sbc_type" default="'rpi'" />
+  <!-- Where the IMU (imu_link) sits on chassis_link. Provisional: the position of an earlier,
+       commented-out IMU in this file, with the board's axes along the robot's (x forward, z up).
+       The real BNO055's mounting on the robot isn't confirmed yet; correct both when it is, or
+       override them, for example imu_xyz:='-0.04 0.02 0.012' imu_rpy:='0 0 0'. -->
+  <xacro:arg name="imu_xyz" default="-0.045 0.02 0.01" />
+  <xacro:arg name="imu_rpy" default="0 0 0" />
   <xacro:property name="package_name" value="remo_description"/>
   <xacro:property name="robot_name" value="remo"/>
@@ -151,9 +157,9 @@
     </xacro:camera_sensor>
   </xacro:if>
-  <!-- IMU
+  <!-- IMU: a BNO055 on the breadboard next to the Teensy, which reads it -->
   <xacro:imu_sensor parent_link="chassis_link"
                     sensor_prop="${sensor_props}">
-    <origin xyz="-0.045 0.02 0.01" rpy="0 0 0" />
-  </xacro:imu_sensor>-->
+    <origin xyz="$(arg imu_xyz)" rpy="$(arg imu_rpy)" />
+  </xacro:imu_sensor>
   <!-- Gazebo -->
   <xacro:gazebo_ros_control robotNamespace="/diffbot">
